Commit message: Differential drive

File: urdf/mir100.urdf.xacro (robot description, xacro)
@@ -2,5 +2,5 @@
 <robot xmlns:xacro="http://www.ros.org/wiki/xacro" name="mir100">
 <xacro:include filename="$(find mir100_description)/urdf/wheel.urdf.xacro" />
-<!--                    Property list                             -->
+<!--                          PROPERTY LIST                         -->
 <!-- Robot's dimensions -->
 <xacro:property name="body_height" value="0.300" />
@@ -14,15 +14,17 @@
 <xacro:property name="base_y_origin_to_castorwheel_origin" value="${base_y_origin_to_wheel_origin}" />
 <!-- Motor wheels -->
-<xacro:property name="wheel_radius" value="0.03" />
+<xacro:property name="motor_wheel_radius" value="0.03" />
+<xacro:property name="motor_wheel_epsilon" value="0.0001" />
+<xacro:property name="castor_wheel_radius" value="0.03" />
 <xacro:property name="wheel_thickness" value="0.03" />
 <xacro:property name="wheel_ext_s2s_distance" value="0.480" />
 <xacro:property name="base_x_origin_to_wheel_origin" value="0.0" />
 <xacro:property name="base_y_origin_to_wheel_origin" value="${(wheel_ext_s2s_distance-wheel_thickness)/2}" />
-<xacro:property name="base_z_origin_to_wheel_origin" value="${wheel_radius-robot_height}" />
+<xacro:property name="base_z_origin_to_wheel_origin" value="${motor_wheel_radius-robot_height}" />
 <!-- All mass in kg-->
 <xacro:property name="motor_wheel_mass" value="1.5" />
 <xacro:property name="castor_wheel_mass" value="1.5" />
 <xacro:property name="body_mass" value="10" />
-<!--                    Material definition                     -->
+<!--                    MATERIAL DEFINITION                         -->
 <material name="black">
 	<color rgba="0 0 0 1"/>
@@ -34,5 +36,5 @@
 	<color rgba="0 0 0.8 1"/>
 </material>
-<!--                    Inertia basic shape macro                     -->
+<!--                    INERTIA MACRO                              -->
 <xacro:macro name="cylinder_inertia" params="m r h">
   <inertia  ixx="${m*(3*r*r+h*h)/12}" ixy = "0" ixz = "0"
@@ -45,5 +47,11 @@
             izz="${m*(x*x+z*z)/12}" />
 </xacro:macro>
-<!--                    Base footprint                        -->
+<xacro:macro name="default_inertial" params="mass">
+  <inertial>
+    <mass value="${mass}" />
+    <inertia ixx="1.0" ixy="0.0" ixz="0.0" iyy="1.0" iyz="0.0" izz="1.0" />
+  </inertial>
+</xacro:macro>
+<!--                    BASE FOOTPRINT                             -->
 <!-- Link that is on the ground right below base_link origin  -->
 <link name="base_footprint">
@@ -71,5 +79,5 @@
   <child link="base_link" />
 </joint>
-<!--                    Base link                           -->
+<!--                    BASE LINK                                 -->
 <link name="base_link">
 	<visual>
@@ -95,19 +103,19 @@
 	<turnGravityOff>false</turnGravityOff>
 </gazebo>
-<!--                    Motor wheels                        -->
+<!--                    MOTOR WHEELS                             -->
 <wheel lr="left" parent="base_link" translateX="0" translateY="1" flipY="1"/>
 <wheel lr="right" parent="base_link" translateX="0" translateY="-1" flipY="1"/>
-<!--                    Castor wheels                       -->
+<!--                    CASTOR WHEELS                            -->
 <!-- Left front -->
 <link name="left_front_castor_wheel">
-	<visual>
-		<geometry>
-			<sphere radius="${wheel_radius}"/>
-		</geometry>
-		<material name="white"/>
-	</visual>
-  <collision>
-    <geometry>
-      <sphere radius="${wheel_radius}" />
+  <visual>
+    <geometry>
+      <sphere radius="${castor_wheel_radius}"/>
+    </geometry>
+    <material name="white"/>
+  </visual>
+  <collision>
+    <geometry>
+      <sphere radius="${castor_wheel_radius}" />
     </geometry>
   </collision>
@@ -121,19 +129,19 @@
 </link>
 <joint name="base_to_left_front_castor_wheel" type="fixed">
-	<parent link="base_link"/>
-	<child link="left_front_castor_wheel"/>
-	<origin rpy="0 0 0" xyz="${base_x_origin_to_castorwheel_origin} ${base_y_origin_to_castorwheel_origin} ${wheel_radius-robot_height}"/>
+  <parent link="base_link"/>
+  <child link="left_front_castor_wheel"/>
+  <origin rpy="0 0 0" xyz="${base_x_origin_to_castorwheel_origin} ${base_y_origin_to_castorwheel_origin} ${castor_wheel_radius-robot_height}"/>
 </joint>
 <!-- Left rear -->
 <link name="left_rear_castor_wheel">
-	<visual>
-		<geometry>
-			<sphere radius="${wheel_radius}"/>
-		</geometry>
-		<material name="white"/>
-	</visual>
-  <collision>
-    <geometry>
-      <sphere radius="${wheel_radius}" />
+  <visual>
+    <geometry>
+      <sphere radius="${castor_wheel_radius}"/>
+    </geometry>
+    <material name="white"/>
+  </visual>
+  <collision>
+    <geometry>
+      <sphere radius="${castor_wheel_radius}" />
     </geometry>
   </collision>
@@ -147,19 +155,19 @@
 </link>
 <joint name="base_to_left_rear_castor_wheel" type="fixed">
-	<parent link="base_link"/>
-	<child link="left_rear_castor_wheel"/>
-	<origin rpy="0 0 0" xyz="-${base_x_origin_to_castorwheel_origin} ${base_y_origin_to_castorwheel_origin} ${wheel_radius-robot_height}"/>
+  <parent link="base_link"/>
+  <child link="left_rear_castor_wheel"/>
+  <origin rpy="0 0 0" xyz="-${base_x_origin_to_castorwheel_origin} ${base_y_origin_to_castorwheel_origin} ${castor_wheel_radius-robot_height}"/>
 </joint>
 <!-- Right front -->
 <link name="right_front_castor_wheel">
-	<visual>
-		<geometry>
-			<sphere radius="${wheel_radius}"/>
-		</geometry>
-		<material name="white"/>
-	</visual>
-  <collision>
-    <geometry>
-      <sphere radius="${wheel_radius}" />
+  <visual>
+    <geometry>
+      <sphere radius="${castor_wheel_radius}"/>
+    </geometry>
+    <material name="white"/>
+  </visual>
+  <collision>
+    <geometry>
+      <sphere radius="${castor_wheel_radius}" />
     </geometry>
   </collision>
@@ -173,19 +181,19 @@
 </link>
 <joint name="base_to_right_front_castor_wheel" type="fixed">
-	<parent link="base_link"/>
-	<child link="right_front_castor_wheel"/>
-	<origin rpy="0 0 0" xyz="${base_x_origin_to_castorwheel_origin} -${base_y_origin_to_castorwheel_origin} ${wheel_radius-robot_height}"/>
+  <parent link="base_link"/>
+  <child link="right_front_castor_wheel"/>
+  <origin rpy="0 0 0" xyz="${base_x_origin_to_castorwheel_origin} -${base_y_origin_to_castorwheel_origin} ${castor_wheel_radius-robot_height}"/>
 </joint>
 <!-- Left rear -->
 <link name="right_rear_castor_wheel">
-	<visual>
-		<geometry>
-			<sphere radius="${wheel_radius}"/>
-		</geometry>
-		<material name="white"/>
-	</visual>
-  <collision>
-    <geometry>
-      <sphere radius="${wheel_radius}" />
+  <visual>
+    <geometry>
+      <sphere radius="${castor_wheel_radius}"/>
+    </geometry>
+    <material name="white"/>
+  </visual>
+  <collision>
+    <geometry>
+      <sphere radius="${castor_wheel_radius}" />
     </geometry>
   </collision>
@@ -199,84 +207,13 @@
 </link>
 <joint name="base_to_right_rear_castor_wheel" type="fixed">
-	<parent link="base_link"/>
-	<child link="right_rear_castor_wheel"/>
-	<origin rpy="0 0 0" xyz="-${base_x_origin_to_castorwheel_origin} -${base_y_origin_to_castorwheel_origin} ${wheel_radius-robot_height}"/>
-</joint>
-<!--                    Differential drive controller       -->
-<!--
+  <parent link="base_link"/>
+  <child link="right_rear_castor_wheel"/>
+  <origin rpy="0 0 0" xyz="-${base_x_origin_to_castorwheel_origin} -${base_y_origin_to_castorwheel_origin} ${castor_wheel_radius-robot_height}"/>
+</joint>
+<!--                    GAZEBO PLUGIN ROS CONTROL                        -->
 <gazebo>
-    <plugin name="differential_drive_controller" filename="libgazebo_ros_diff_drive.so">
-        <alwaysOn>true</alwaysOn>
-        <updateRate>40</updateRate>
-        <legacyMode>false</legacyMode>
-        <leftJoint>base_right_wheel_joint</leftJoint>
-        <rightJoint>base_left_wheel_joint</rightJoint>
-        <wheelSeparation>${wheel_ext_s2s_distance-wheel_thickness}</wheelSeparation>
-        <wheelDiameter>${2*wheel_radius}</wheelDiameter>
-        <torque>5</torque>
-        <commandTopic>cmd_vel</commandTopic>
-        <odometryTopic>odom</odometryTopic>
-        <odometryFrame>odom</odometryFrame>
-        <robotBaseFrame>base_link</robotBaseFrame>
-        <publishWheelTF>false</publishWheelTF>
-        <publishWheelJointState>false</publishWheelJointState>
-        <rosDebugLevel>na</rosDebugLevel>
-        <wheelAcceleration>0</wheelAcceleration>
-        <wheelTorque>5</wheelTorque>
-        <odometrySource>world</odometrySource>
-        <publishTf>1</publishTf>
-    </plugin>
+  <plugin name="gazebo_ros_control" filename="libgazebo_ros_control.so">
+    <robotNamespace>/</robotNamespace>
+  </plugin>
 </gazebo>
--->
-<!--
-  <gazebo>
-    <plugin name="differential_drive_controller" filename="libgazebo_ros_diff_drive.so">
-      <rosDebugLevel>Debug</rosDebugLevel>
-      <publishWheelTF>false</publishWheelTF>
-      <robotNamespace>/</robotNamespace>
-      <publishTf>1</publishTf>
-      <publishWheelJointState>false</publishWheelJointState>
-      <alwaysOn>true</alwaysOn>
-      <updateRate>100.0</updateRate>
-      <leftJoint>front_left_wheel_joint</leftJoint>
-      <rightJoint>front_right_wheel_joint</rightJoint>
-      <wheelSeparation>${wheel_ext_s2s_distance-wheel_thickness}</wheelSeparation>
-      <wheelDiameter>${2*wheel_radius}</wheelDiameter>
-      <legacyMode>true</legacyMode>
-      <odometrySource>world</odometrySource>
-      <broadcastTF>1</broadcastTF>
-      <wheelTorque>30</wheelTorque>
-      <wheelAcceleration>1.8</wheelAcceleration>
-      <commandTopic>cmd_vel</commandTopic>
-      <odometryFrame>odom</odometryFrame>
-      <odometryTopic>odom</odometryTopic>
-      <robotBaseFrame>base_footprint</robotBaseFrame>
-    </plugin>
-</gazebo>
--->
-  <!-- Gazebo plugin for ROS Control -->
-  <gazebo>
-    <plugin name="gazebo_ros_control" filename="libgazebo_ros_control.so">
-      <robotNamespace>/</robotNamespace>
-    </plugin>
-</gazebo>
-  <!--                GAZEBO RELATED PART                             -->
-  <!-- ROS Control plugin for Gazebo
-  <gazebo>
-    <plugin name="gazebo_ros_control" filename="libgazebo_ros_control.so">
-      <robotNamespace>/mir100_model</robotNamespace>
-    </plugin>
-  </gazebo>
--->
-  <!-- transmission
-  <transmission name="base_to_right_wheel_trans">
-    <type>transmission_interface/SimpleTransmission</type>
-    <actuator name="motor1">
-      <mechanicalReduction>1</mechanicalReduction>
-    </actuator>
-    <joint name="base_to_right_wheel">
-      <hardwareInterface>EffortJointInterface</hardwareInterface>
-    </joint>
-  </transmission>
--->
 </robot>

File: urdf/wheel.urdf.xacro (robot description, xacro)
@@ -6,5 +6,5 @@
         <origin xyz="0 0 0" rpy="${flipY*pi/2} 0  0 " />
         <geometry>
-          <cylinder length="${wheel_thickness}" radius="${wheel_radius}" />
+          <cylinder length="${wheel_thickness}" radius="${motor_wheel_radius+motor_wheel_epsilon}" />
         </geometry>
         <material name="DarkGray" />
@@ -13,5 +13,5 @@
         <origin xyz="0 0 0" rpy="${flipY*pi/2} 0 0 " />
         <geometry>
-          <cylinder length="${wheel_thickness}" radius="${wheel_radius}" />
+          <cylinder length="${wheel_thickness}" radius="${motor_wheel_radius+motor_wheel_epsilon}" />
         </geometry>
       </collision>
@@ -19,5 +19,5 @@
         <mass value="${motor_wheel_mass}" />
         <origin xyz="0 0 0" />
-        <cylinder_inertia  m="${motor_wheel_mass}" r="${wheel_radius}" h="${wheel_thickness}" />
+        <cylinder_inertia  m="${motor_wheel_mass}" r="${motor_wheel_radius}" h="${wheel_thickness}" />
       </inertial>
     </link>
@@ -27,5 +27,4 @@
       <kp  value="10000000.0" />
       <kd  value="1.0" />
-      <fdir1 value="1 0 0"/>
       <material>Gazebo/Grey</material>
       <turnGravityOff>false</turnGravityOff>
@@ -45,5 +44,5 @@
       </actuator>
       <joint name="${lr}_wheel_joint">
-        <hardwareInterface>VelocityJointInterface</hardwareInterface>
+        <hardwareInterface>hardware_interface/VelocityJointInterface</hardwareInterface>
       </joint>
     </transmission>

Commit message: Merge camera and MIR100

File: urdf/mir100.urdf.xacro (robot description, xacro)
@@ -25,5 +25,5 @@
 <xacro:property name="motor_wheel_mass" value="1.5" />
 <xacro:property name="castor_wheel_mass" value="1.5" />
-<xacro:property name="body_mass" value="10" />
+<xacro:property name="body_mass" value="67" />
 <!--                    MATERIAL DEFINITION                         -->
 <material name="black">
@@ -214,5 +214,5 @@
 <gazebo>
   <plugin name="gazebo_ros_control" filename="libgazebo_ros_control.so">
-    <robotNamespace>/</robotNamespace>
+    <!-- no robotNamespace>/</robotNamespace> for multi-robobt integration -->
   </plugin>
 </gazebo>

Commit message: alvar tag integration

File: urdf/mir100.urdf.xacro (robot description, xacro)
@@ -4,10 +4,8 @@
 <!--                          PROPERTY LIST                         -->
 <!-- Robot's dimensions -->
-<xacro:property name="body_height" value="0.300" />
+<xacro:property name="body_height" value="0.270" />
 <xacro:property name="body_width" value="0.550" />
 <xacro:property name="body_len" value="0.900" />
 <xacro:property name="robot_height" value="0.350" />
-<!-- Mathematical constant -->
-<xacro:property name="deg2rad" value="0.017453293" />
 <!-- Castor wheels -->
 <xacro:property name="base_x_origin_to_castorwheel_origin" value="0.310" />
@@ -22,8 +20,14 @@
 <xacro:property name="base_y_origin_to_wheel_origin" value="${(wheel_ext_s2s_distance-wheel_thickness)/2}" />
 <xacro:property name="base_z_origin_to_wheel_origin" value="${motor_wheel_radius-robot_height}" />
+<!-- Differential driver parameters -->
+<xacro:property name="wheel_separation" value="${(wheel_ext_s2s_distance-wheel_thickness)}" />
+<xacro:property name="wheel_radius" value="${motor_wheel_epsilon + motor_wheel_epsilon}" />
 <!-- All mass in kg-->
-<xacro:property name="motor_wheel_mass" value="1.5" />
-<xacro:property name="castor_wheel_mass" value="1.5" />
+<xacro:property name="motor_wheel_mass" value="1" />
+<xacro:property name="castor_wheel_mass" value="1" />
 <xacro:property name="body_mass" value="67" />
+<!-- Friction-->
+<xacro:property name="coulomb_friction_first_direction" value="0.01" />
+<xacro:property name="coulomb_friction_second_direction" value="0.01" />
 <!--                    MATERIAL DEFINITION                         -->
 <material name="black">
@@ -50,5 +54,7 @@
   <inertial>
     <mass value="${mass}" />
-    <inertia ixx="1.0" ixy="0.0" ixz="0.0" iyy="1.0" iyz="0.0" izz="1.0" />
+    <inertia ixx="1.0" ixy="0.0" ixz="0.0"
+             iyy="1.0" iyz="0.0"
+             izz="1.0" />
   </inertial>
 </xacro:macro>
@@ -74,17 +80,16 @@
   <turnGravityOff>false</turnGravityOff>
 </gazebo>
-<joint name="base_footprint_joint" type="fixed">
-  <origin xyz="0 0 ${robot_height}" rpy="0 0 0" />
-  <parent link="base_footprint"/>
-  <child link="base_link" />
-</joint>
 <!--                    BASE LINK                                 -->
 <link name="base_link">
 	<visual>
+      <geometry>
+        <mesh filename="package://mir100_description/meshes/body.dae"/>
+      </geometry>
+<!--
 			<geometry>
 				<box size="${body_len} ${body_width} ${body_height}"/>
 			</geometry>
+-->
 			<origin rpy="0 0 0" xyz="0 0 -${body_height/2}"/>
-		<material name="white"/>
 	</visual>
 	<collision>
@@ -100,4 +105,9 @@
 	</inertial>
 </link>
+<joint name="base_footprint_joint" type="fixed">
+  <origin xyz="0 0 ${robot_height}" rpy="0 0 0" />
+  <parent link="base_footprint"/>
+  <child link="base_link" />
+</joint>
 <gazebo reference="base_link">
 	<turnGravityOff>false</turnGravityOff>
@@ -120,11 +130,5 @@
     </geometry>
   </collision>
-  <inertial>
-    <mass value="${castor_wheel_mass}" />
-    <origin xyz="0 0 0" />
-    <inertia ixx="0.001" ixy="0.0" ixz="0.0"
-             iyy="0.001" iyz="0.0"
-             izz="0.001" />
-  </inertial>
+  <xacro:default_inertial mass="${castor_wheel_mass}"/>
 </link>
 <joint name="base_to_left_front_castor_wheel" type="fixed">
@@ -146,11 +150,5 @@
     </geometry>
   </collision>
-  <inertial>
-    <mass value="${castor_wheel_mass}" />
-    <origin xyz="0 0 0" />
-    <inertia ixx="0.001" ixy="0.0" ixz="0.0"
-             iyy="0.001" iyz="0.0"
-             izz="0.001" />
-  </inertial>
+  <xacro:default_inertial mass="${castor_wheel_mass}"/>
 </link>
 <joint name="base_to_left_rear_castor_wheel" type="fixed">
@@ -172,11 +170,5 @@
     </geometry>
   </collision>
-  <inertial>
-    <mass value="${castor_wheel_mass}" />
-    <origin xyz="0 0 0" />
-    <inertia ixx="0.001" ixy="0.0" ixz="0.0"
-             iyy="0.001" iyz="0.0"
-             izz="0.001" />
-  </inertial>
+  <xacro:default_inertial mass="${castor_wheel_mass}"/>
 </link>
 <joint name="base_to_right_front_castor_wheel" type="fixed">
@@ -198,11 +190,5 @@
     </geometry>
   </collision>
-  <inertial>
-    <mass value="${castor_wheel_mass}" />
-    <origin xyz="0 0 0" />
-    <inertia ixx="0.001" ixy="0.0" ixz="0.0"
-             iyy="0.001" iyz="0.0"
-             izz="0.001" />
-  </inertial>
+  <xacro:default_inertial mass="${castor_wheel_mass}"/>
 </link>
 <joint name="base_to_right_rear_castor_wheel" type="fixed">
@@ -211,4 +197,30 @@
   <origin rpy="0 0 0" xyz="-${base_x_origin_to_castorwheel_origin} -${base_y_origin_to_castorwheel_origin} ${castor_wheel_radius-robot_height}"/>
 </joint>
+<!--                    GAZEBO FRICTION                                  -->
+<gazebo reference="base_link">
+  <mu1>${coulomb_friction_first_direction}</mu1>
+  <mu2>${coulomb_friction_second_direction}</mu2>
+  <material>Gazebo/white</material>
+</gazebo>
+<gazebo reference="left_front_castor_wheel">
+  <mu1>${coulomb_friction_first_direction}</mu1>
+  <mu2>${coulomb_friction_second_direction}</mu2>
+  <material>Gazebo/Black</material>
+</gazebo>
+<gazebo reference="right_front_castor_wheel">
+  <mu1>${coulomb_friction_first_direction}</mu1>
+  <mu2>${coulomb_friction_second_direction}</mu2>
+  <material>Gazebo/Black</material>
+</gazebo>
+<gazebo reference="left_rear_castor_wheel">
+  <mu1>${coulomb_friction_first_direction}</mu1>
+  <mu2>${coulomb_friction_second_direction}</mu2>
+  <material>Gazebo/Black</material>
+</gazebo>
+<gazebo reference="right_rear_castor_wheel">
+  <mu1>${coulomb_friction_first_direction}</mu1>
+  <mu2>${coulomb_friction_second_direction}</mu2>
+  <material>Gazebo/Black</material>
+</gazebo>
 <!--                    GAZEBO PLUGIN ROS CONTROL                        -->
 <gazebo>

File: urdf/wheel.urdf.xacro (robot description, xacro)
@@ -27,4 +27,5 @@
       <kp  value="10000000.0" />
       <kd  value="1.0" />
+      <fdir1 value="1 0 0"/>
       <material>Gazebo/Grey</material>
       <turnGravityOff>false</turnGravityOff>
